Commit message: update robot to have only 3 joints

File: robot/simple.urdf (robot description, URDF)
Before this commit: robot simple, 7 links, 6 joints
Links:
- removed link dummy_elbow
- added link arm_link00; collision cylinder length=0.3 radius=0.02; visual cylinder length=0.3 radius=0.02
- link arm_link0: geometry collision cylinder length=0.5 radius=0.02; visual cylinder length=0.5 radius=0.02
- link arm_link1: geometry collision cylinder length=0.5 radius=0.02; visual cylinder length=0.5 radius=0.02
Joints:
- removed joint elbow_0
- removed joint elbow_1
- added joint elbow: type revolute, parent arm_link0, child arm_link1, origin xyz=0 0.5 0 rpy=0 0 0, axis 0 0 1, limit lower=-0 upper=0 effort=1000.0 velocity=1000.0
- added joint shoulder_visual_joint: type fixed, parent base_link, child arm_link00, origin xyz=0 0 0 rpy=0 0 0, axis 0 0 1, limit lower=-1.5707963267948966 upper=1.5707963267948966 effort=1000.0 velocity=1000.0
- joint dummy_ee: origin xyz=0.4318 0 0 rpy=0 0 0 -> xyz=0.5 0 0 rpy=0 0 0
- joint shoulder_lift: origin xyz=0 0 0 rpy=1.5707963267948966 0 0 -> xyz=0 0 0.3 rpy=1.5707963267948966 0 0

File: robot/simple.xacro (robot description, xacro)
@@ -11,5 +11,6 @@
     <color rgba="1 0 0 1"/>
   </material>
-  <xacro:property name="link_length" value="0.4318" />
+  <xacro:property name="link_1_length" value = "0.3" />
+  <xacro:property name="link_length" value="0.5" />
   <xacro:property name="dummy_link_length" value="0.1" />
   <xacro:property name="link_radius" value="0.02" />
@@ -29,5 +30,5 @@
   <link name="dummy_link0">
     <visual>
-      <origin rpy="${pi/2} 0 0" xyz="0 0 0"/>
+      <origin rpy="${pi/2} 0 0" xyz="0 0 ${link_1_length}"/>
       <geometry>
         <cylinder length="${dummy_link_length}" radius="${link_radius}"/>
@@ -44,4 +45,26 @@
     <parent link="base_link"/>
     <child link="dummy_link0"/>
+    <origin rpy="0 0 0" xyz="0 0 0"/>
+    <axis xyz="0 0 1"/>
+    <limit effort="1000.0" lower="-${pi/2}" upper="${pi/2}" velocity="1000.0"/>
+  </joint>
+  <link name="arm_link00">
+    <visual>
+      <origin rpy="$0 0 0" xyz="0 0 ${link_1_length/2}"/>
+      <geometry>
+        <cylinder length="${link_1_length}" radius="${link_radius}"/>
+      </geometry>
+      <material name="blue"/>
+    </visual>
+    <collision>
+      <origin rpy="$0 0 0" xyz="0 0 ${link_1_length/2}"/>
+      <geometry>
+        <cylinder length="${link_1_length}" radius="${link_radius}"/>
+      </geometry>
+    </collision>
+  </link>
+  <joint name="shoulder_visual_joint" type="fixed">
+    <parent link="base_link"/>
+    <child link="arm_link00"/>
     <origin rpy="0 0 0" xyz="0 0 0"/>
     <axis xyz="0 0 1"/>
@@ -72,9 +95,9 @@
     <child link="arm_link0"/>
     <!-- <origin xyz="0 0 0"/> -->
-    <origin rpy="${pi/2} 0 0" xyz="0 0 0"/>
+    <origin rpy="${pi/2} 0 0" xyz="0 0 ${link_1_length}"/>
     <axis xyz="0 0 1"/>
     <limit effort="1000.0" lower="-${pi}" upper="${0}" velocity="1000.0"/>
   </joint>
-  <link name="dummy_elbow">
+  <!-- <link name="dummy_elbow">
     <visual>
       <origin rpy="0 0 0" xyz="0 0 0"/>
@@ -84,13 +107,12 @@
       <material name="red"/>
     </visual>
-  </link>
-  <joint name="elbow_0" type="revolute">
+  </link> -->
+  <!-- <joint name="elbow_0" type="revolute">
     <parent link="arm_link0"/>
     <child link="dummy_elbow"/>
-    <!-- <origin xyz="0 0 0"/> -->
     <origin rpy="-${pi/2} 0 0" xyz="0 ${link_length} 0"/>
     <axis xyz="0 0 1"/>
     <limit effort="1000.0" lower="-${0}" upper="${0}" velocity="1000.0"/>
-  </joint>
+  </joint> -->
   <link name="arm_link1">
     <visual>
@@ -108,5 +130,12 @@
     </collision>
   </link>
-  <joint name="elbow_1" type="revolute">
+  <joint name="elbow" type="revolute">
+    <parent link="arm_link0"/>
+    <child link="arm_link1"/>
+    <origin rpy="0 0 0" xyz="0 ${link_length} 0"/>
+    <axis xyz="0 0 1"/>
+    <limit effort="1000.0" lower="-${0}" upper="${0}" velocity="1000.0"/>
+  </joint>
+  <!-- <joint name="elbow_1" type="revolute">
     <parent link="dummy_elbow"/>
     <child link="arm_link1"/>
@@ -114,8 +143,8 @@
     <axis xyz="0 0 1"/>
     <limit effort="1000.0" lower="-${pi}" upper="${0}" velocity="1000.0"/>
-  </joint>
+  </joint> -->
   <link name="dummy_elbow2">
     <visual>
-      <origin rpy="0 0 0" xyz="0 0 0"/>
+      <origin rpy="{pi/2} 0 0" xyz="0 0 0"/>
       <geometry>
         <cylinder length="${dummy_link_length}" radius="${link_radius}"/>
